File: reader.sch (EAGLE design)
At the start: 14 parts, among them J1 RJ11-6PTH, J2 AVR_SPI_PRG_6NS

Commit message: Add a switch transistor to drive the speaker
Parts:
- added R6: 160R, SparkFun-Passives:RESISTOR0805-RES
- added T1: BC547, transistor:BC547
- R4: value 66R -> 1K8
Connections:
- removed net N$9: JP2.3, R4.2
- new net N$4: R4.2, T1.B
- new net N$5: R6.1, T1.E
- new net N$7: JP2.3, R6.2
- net VCC: now also T1.C
Other:
- moved on the sheet: R4
Changed lines of the file:
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@@
 <part name="SUPPLY4" library="SparkFun-Aesthetics" deviceset="VCC" device=""/>
 <part name="R5" library="SparkFun-Passives" deviceset="RESISTOR" device="0805-RES" value="4K7"/>
-<part name="R4" library="SparkFun-Passives" deviceset="RESISTOR" device="0805-RES" value="66R"/>
+<part name="R4" library="SparkFun-Passives" deviceset="RESISTOR" device="0805-RES" value="1K8"/>
 <part name="J2" library="SparkFun-Connectors" deviceset="AVR_SPI_PRG_6" device="NS"/>
 <part name="SUPPLY5" library="SparkFun-Aesthetics" deviceset="VCC" device=""/>
@@
 <part name="SP1" library="buzzer" deviceset="AL23P" device=""/>
 <part name="JP2" library="jumper" deviceset="JP2E" device=""/>
+<part name="T1" library="transistor" deviceset="BC547" device=""/>
+<part name="P+1" library="supply1" deviceset="VCC" device=""/>
+<part name="R6" library="SparkFun-Passives" deviceset="RESISTOR" device="0805-RES" value="160R"/>
 </parts>
 <sheets>
@@
 <instance part="SUPPLY4" gate="G$1" x="-27.94" y="-35.56"/>
 <instance part="R5" gate="G$1" x="-78.74" y="5.08"/>
-<instance part="R4" gate="G$1" x="-10.16" y="45.72"/>
+<instance part="R4" gate="G$1" x="-12.7" y="40.64"/>
 <instance part="J2" gate="G$1" x="-78.74" y="-48.26"/>
 <instance part="SUPPLY5" gate="G$1" x="-53.34" y="-35.56"/>
@@
 <instance part="SP1" gate="G$1" x="60.96" y="43.18" rot="R270"/>
 <instance part="JP2" gate="1" x="2.54" y="55.88"/>
+<instance part="T1" gate="G$1" x="-2.54" y="40.64" rot="MR180"/>
+<instance part="P+1" gate="VCC" x="5.08" y="38.1"/>
+<instance part="R6" gate="G$1" x="7.62" y="45.72"/>
 </instances>
 <busses>
@@
 <wire x1="-68.58" y1="-45.72" x2="-53.34" y2="-45.72" width="0.1524" layer="91"/>
 <wire x1="-53.34" y1="-45.72" x2="-53.34" y2="-35.56" width="0.1524" layer="91"/>
+</segment>
+<segment>
+<pinref part="T1" gate="G$1" pin="C"/>
+<wire x1="0" y1="35.56" x2="0" y2="33.02" width="0.1524" layer="91"/>
+<wire x1="0" y1="33.02" x2="5.08" y2="33.02" width="0.1524" layer="91"/>
+<pinref part="P+1" gate="VCC" pin="VCC"/>
+<wire x1="5.08" y1="33.02" x2="5.08" y2="35.56" width="0.1524" layer="91"/>
 </segment>
 </net>
@@
 <segment>
 <pinref part="R4" gate="G$1" pin="1"/>
-<wire x1="-15.24" y1="45.72" x2="-25.4" y2="45.72" width="0.1524" layer="91"/>
-<label x="-25.4" y="45.72" size="1.778" layer="95"/>
+<wire x1="-17.78" y1="40.64" x2="-30.48" y2="40.64" width="0.1524" layer="91"/>
+<label x="-30.48" y="40.64" size="1.778" layer="95"/>
 </segment>
 <segment>
@@
 <wire x1="68.58" y1="10.16" x2="81.28" y2="10.16" width="0.1524" layer="91"/>
 <label x="68.58" y="10.16" size="1.778" layer="95"/>
-</segment>
-</net>
-<net name="N$9" class="0">
-<segment>
-<pinref part="R4" gate="G$1" pin="2"/>
-<wire x1="-5.08" y1="45.72" x2="5.08" y2="45.72" width="0.1524" layer="91"/>
-<wire x1="5.08" y1="45.72" x2="5.08" y2="53.34" width="0.1524" layer="91"/>
-<pinref part="JP2" gate="1" pin="3"/>
 </segment>
 </net>
@@
 </segment>
 </net>
+<net name="N$4" class="0">
+<segment>
+<pinref part="R4" gate="G$1" pin="2"/>
+<pinref part="T1" gate="G$1" pin="B"/>
+<wire x1="-7.62" y1="40.64" x2="-5.08" y2="40.64" width="0.1524" layer="91"/>
+</segment>
+</net>
+<net name="N$5" class="0">
+<segment>
+<pinref part="T1" gate="G$1" pin="E"/>
+<wire x1="0" y1="45.72" x2="2.54" y2="45.72" width="0.1524" layer="91"/>
+<pinref part="R6" gate="G$1" pin="1"/>
+</segment>
+</net>
+<net name="N$7" class="0">
+<segment>
+<wire x1="12.7" y1="45.72" x2="12.7" y2="53.34" width="0.1524" layer="91"/>
+<pinref part="JP2" gate="1" pin="3"/>
+<wire x1="12.7" y1="53.34" x2="5.08" y2="53.34" width="0.1524" layer="91"/>
+<pinref part="R6" gate="G$1" pin="2"/>
+</segment>
+</net>

Commit message: Swap SPEAKER and BLUE_LED, reorganize components
Connections:
- net BLUE_LED: now also U$1.PA0/PCINT0/ADC0/AREF/MISO; no longer U$1.PA3/PCINT3/ADC3/AIN10/TOCC2/T0/XCK0/SCK
- net SPEAKER: now also U$1.PA3/PCINT3/ADC3/AIN10/TOCC2/T0/XCK0/SCK; no longer U$1.PA0/PCINT0/ADC0/AREF/MISO
Changed lines of the file:
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@@
 </variantdefs>
 <classes>
-<class number="0" name="default" width="0.6096" drill="0">
+<class number="0" name="default" width="0.3302" drill="1">
 </class>
 </classes>
@@
 </segment>
 <segment>
-<pinref part="U$1" gate="G$1" pin="PA3/PCINT3/ADC3/AIN10/TOCC2/T0/XCK0/SCK"/>
-<wire x1="68.58" y1="2.54" x2="81.28" y2="2.54" width="0.1524" layer="91"/>
-<label x="68.58" y="2.54" size="1.778" layer="95"/>
+<pinref part="U$1" gate="G$1" pin="PA0/PCINT0/ADC0/AREF/MISO"/>
+<wire x1="68.58" y1="10.16" x2="81.28" y2="10.16" width="0.1524" layer="91"/>
+<label x="68.58" y="10.16" size="1.778" layer="95"/>
 </segment>
 </net>
@@
 </segment>
 <segment>
-<pinref part="U$1" gate="G$1" pin="PA0/PCINT0/ADC0/AREF/MISO"/>
-<wire x1="68.58" y1="10.16" x2="81.28" y2="10.16" width="0.1524" layer="91"/>
-<label x="68.58" y="10.16" size="1.778" layer="95"/>
-</segment>
-</net>
+<pinref part="U$1" gate="G$1" pin="PA3/PCINT3/ADC3/AIN10/TOCC2/T0/XCK0/SCK"/>
+<wire x1="68.58" y1="2.54" x2="81.28" y2="2.54" width="0.1524" layer="91"/>
+<label x="68.58" y="2.54" size="1.778" layer="95"/>
+</segment>
+</net>

Commit message: [WIP] Manually route few connectors on the board
Parts:
- renumbered LD1 to LED2, U$1 to U1
Changed lines of the file:
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@@
 </variantdefs>
 <classes>
-<class number="0" name="default" width="0.3302" drill="1">
+<class number="0" name="default" width="0.3302" drill="0.381">
 </class>
 </classes>
 <parts>
-<part name="U$1" library="attiny841" deviceset="TINY841" device=""/>
+<part name="U1" library="attiny841" deviceset="TINY841" device=""/>
 <part name="FRAME1" library="frames" deviceset="A4L-LOC" device=""/>
 <part name="SUPPLY1" library="SparkFun-Aesthetics" deviceset="VCC" device=""/>
@@
 <part name="LED1" library="led" deviceset="LED" device="3MM" value="BLUE"/>
 <part name="R3" library="SparkFun-Passives" deviceset="RESISTOR" device="0805-RES" value="680R"/>
-<part name="LD1" library="led" deviceset="DUOLED-RY-C" device="" value="STATUS"/>
+<part name="LED2" library="led" deviceset="DUOLED-RY-C" device="" value="STATUS"/>
 <part name="J1" library="SparkFun-Connectors" deviceset="RJ11-6" device="PTH"/>
 <part name="SUPPLY3" library="SparkFun-Aesthetics" deviceset="VCC" device=""/>
@@
 </plain>
 <instances>
-<instance part="U$1" gate="G$1" x="10.16" y="5.08"/>
+<instance part="U1" gate="G$1" x="10.16" y="5.08"/>
 <instance part="FRAME1" gate="G$1" x="-124.46" y="-81.28"/>
 <instance part="SUPPLY1" gate="G$1" x="-83.82" y="17.78"/>
@@
 <instance part="LED1" gate="G$1" x="58.42" y="55.88" rot="R90"/>
 <instance part="R3" gate="G$1" x="45.72" y="55.88"/>
-<instance part="LD1" gate="G$1" x="60.96" y="73.66" rot="R180"/>
+<instance part="LED2" gate="G$1" x="60.96" y="73.66" rot="R180"/>
 <instance part="J1" gate="G$1" x="-76.2" y="73.66" rot="MR180"/>
 <instance part="SUPPLY3" gate="G$1" x="-55.88" y="78.74"/>
@@
 </segment>
 <segment>
-<pinref part="U$1" gate="G$1" pin="VCC"/>
+<pinref part="U1" gate="G$1" pin="VCC"/>
 <pinref part="SUPPLY1" gate="G$1" pin="VCC"/>
 <wire x1="-48.26" y1="12.7" x2="-83.82" y2="12.7" width="0.1524" layer="91"/>
@@
 </segment>
 <segment>
-<pinref part="J1" gate="G$1" pin="2"/>
-<wire x1="-71.12" y1="76.2" x2="-55.88" y2="76.2" width="0.1524" layer="91"/>
-<pinref part="SUPPLY3" gate="G$1" pin="VCC"/>
-<wire x1="-55.88" y1="76.2" x2="-55.88" y2="78.74" width="0.1524" layer="91"/>
-</segment>
-<segment>
 <pinref part="JP1" gate="G$1" pin="8"/>
 <wire x1="-2.54" y1="-58.42" x2="-27.94" y2="-58.42" width="0.1524" layer="91"/>
@@
 <pinref part="P+1" gate="VCC" pin="VCC"/>
 <wire x1="5.08" y1="33.02" x2="5.08" y2="35.56" width="0.1524" layer="91"/>
+</segment>
+<segment>
+<pinref part="J1" gate="G$1" pin="2"/>
+<pinref part="SUPPLY3" gate="G$1" pin="VCC"/>
+<wire x1="-71.12" y1="76.2" x2="-55.88" y2="76.2" width="0.1524" layer="91"/>
+<wire x1="-55.88" y1="76.2" x2="-55.88" y2="78.74" width="0.1524" layer="91"/>
 </segment>
 </net>
@@
 <wire x1="78.74" y1="55.88" x2="78.74" y2="73.66" width="0.1524" layer="91"/>
 <junction x="78.74" y="55.88"/>
-<pinref part="LD1" gate="G$1" pin="C"/>
+<pinref part="LED2" gate="G$1" pin="C"/>
 <wire x1="78.74" y1="73.66" x2="63.5" y2="73.66" width="0.1524" layer="91"/>
 <pinref part="SP1" gate="G$1" pin="2"/>
 </segment>
 <segment>
-<pinref part="U$1" gate="G$1" pin="GND"/>
+<pinref part="U1" gate="G$1" pin="GND"/>
 <pinref part="GND1" gate="1" pin="GND"/>
 <wire x1="68.58" y1="12.7" x2="91.44" y2="12.7" width="0.1524" layer="91"/>
@@
 <pinref part="R1" gate="G$1" pin="1"/>
 <wire x1="60.96" y1="66.04" x2="50.8" y2="66.04" width="0.1524" layer="91"/>
-<pinref part="LD1" gate="G$1" pin="AR"/>
+<pinref part="LED2" gate="G$1" pin="AR"/>
 </segment>
 </net>
@@
 <pinref part="R2" gate="G$1" pin="1"/>
 <wire x1="60.96" y1="81.28" x2="50.8" y2="81.28" width="0.1524" layer="91"/>
-<pinref part="LD1" gate="G$1" pin="AY"/>
+<pinref part="LED2" gate="G$1" pin="AY"/>
 </segment>
 </net>
 <net name="RED_LED" class="0">
 <segment>
-<pinref part="U$1" gate="G$1" pin="PB0/PCINT8/ADC11/XTAL1/CLKI"/>
+<pinref part="U1" gate="G$1" pin="PB0/PCINT8/ADC11/XTAL1/CLKI"/>
 <wire x1="-63.5" y1="10.16" x2="-48.26" y2="10.16" width="0.1524" layer="91"/>
 <label x="-63.5" y="10.16" size="1.778" layer="95"/>
@@
 <net name="GREEN_LED" class="0">
 <segment>
-<pinref part="U$1" gate="G$1" pin="PB2/PCINT10/ADC8/CLKO/TOCC7/ICP2/RXD0"/>
+<pinref part="U1" gate="G$1" pin="PB2/PCINT10/ADC8/CLKO/TOCC7/ICP2/RXD0"/>
 <wire x1="-63.5" y1="2.54" x2="-48.26" y2="2.54" width="0.1524" layer="91"/>
 <label x="-63.5" y="2.54" size="1.778" layer="95"/>
@@
 </segment>
 <segment>
-<pinref part="U$1" gate="G$1" pin="PA2/PCINT2/ADC2/AIN01/TOCC1/RXD0/SS"/>
+<pinref part="U1" gate="G$1" pin="PA2/PCINT2/ADC2/AIN01/TOCC1/RXD0/SS"/>
 <wire x1="68.58" y1="5.08" x2="81.28" y2="5.08" width="0.1524" layer="91"/>
 <label x="68.58" y="5.08" size="1.778" layer="95"/>
@@
 </segment>
 <segment>
-<pinref part="U$1" gate="G$1" pin="PA1/PCINT1/ADC1/AIN00/TOCC0/TXD0/MOSI"/>
+<pinref part="U1" gate="G$1" pin="PA1/PCINT1/ADC1/AIN00/TOCC0/TXD0/MOSI"/>
 <wire x1="68.58" y1="7.62" x2="81.28" y2="7.62" width="0.1524" layer="91"/>
 <label x="68.58" y="7.62" size="1.778" layer="95"/>
@@
 </segment>
 <segment>
-<pinref part="U$1" gate="G$1" pin="PA7/PCINT7/ADC7/TOCC6/ICP1/TXD0/SS"/>
+<pinref part="U1" gate="G$1" pin="PA7/PCINT7/ADC7/TOCC6/ICP1/TXD0/SS"/>
 <wire x1="-48.26" y1="0" x2="-63.5" y2="0" width="0.1524" layer="91"/>
 <label x="-60.96" y="0" size="1.778" layer="95"/>
@@
 </segment>
 <segment>
-<pinref part="U$1" gate="G$1" pin="PA4/PCINT4/ADC4/AIN11/TOCC3/T1/RXD1/SCL/SCK"/>
+<pinref part="U1" gate="G$1" pin="PA4/PCINT4/ADC4/AIN11/TOCC3/T1/RXD1/SCL/SCK"/>
 <wire x1="68.58" y1="0" x2="81.28" y2="0" width="0.1524" layer="91"/>
 <label x="68.58" y="0" size="1.778" layer="95"/>
@@
 </segment>
 <segment>
-<pinref part="U$1" gate="G$1" pin="PA6/PCINT6/ADC6/ACO1/TOCC5/XCK1/SDA/MOSI"/>
+<pinref part="U1" gate="G$1" pin="PA6/PCINT6/ADC6/ACO1/TOCC5/XCK1/SDA/MOSI"/>
 <wire x1="-48.26" y1="-2.54" x2="-63.5" y2="-2.54" width="0.1524" layer="91"/>
 <label x="-60.96" y="-2.54" size="1.778" layer="95"/>
@@
 </segment>
 <segment>
-<pinref part="U$1" gate="G$1" pin="PA5/PCINT5/ADC5/ACO0/TOCC4/T2/TXD1/MISO"/>
+<pinref part="U1" gate="G$1" pin="PA5/PCINT5/ADC5/ACO0/TOCC4/T2/TXD1/MISO"/>
 <wire x1="68.58" y1="-2.54" x2="81.28" y2="-2.54" width="0.1524" layer="91"/>
 <label x="68.58" y="-2.54" size="1.778" layer="95"/>
@@
 </segment>
 <segment>
-<pinref part="U$1" gate="G$1" pin="PB1/PCINT9/ADC10/XTAL2/INT0"/>
+<pinref part="U1" gate="G$1" pin="PB1/PCINT9/ADC10/XTAL2/INT0"/>
 <wire x1="-48.26" y1="7.62" x2="-63.5" y2="7.62" width="0.1524" layer="91"/>
 <label x="-63.5" y="7.62" size="1.778" layer="95"/>
@@
 </segment>
 <segment>
-<pinref part="U$1" gate="G$1" pin="PB3/PCINT11/ADC9/RESET/DW"/>
+<pinref part="U1" gate="G$1" pin="PB3/PCINT11/ADC9/RESET/DW"/>
 <wire x1="-48.26" y1="5.08" x2="-73.66" y2="5.08" width="0.1524" layer="91"/>
 <pinref part="R5" gate="G$1" pin="2"/>
@@
 </segment>
 <segment>
-<pinref part="U$1" gate="G$1" pin="PA0/PCINT0/ADC0/AREF/MISO"/>
+<pinref part="U1" gate="G$1" pin="PA0/PCINT0/ADC0/AREF/MISO"/>
 <wire x1="68.58" y1="10.16" x2="81.28" y2="10.16" width="0.1524" layer="91"/>
 <label x="68.58" y="10.16" size="1.778" layer="95"/>
@@
 </segment>
 <segment>
-<pinref part="U$1" gate="G$1" pin="PA3/PCINT3/ADC3/AIN10/TOCC2/T0/XCK0/SCK"/>
+<pinref part="U1" gate="G$1" pin="PA3/PCINT3/ADC3/AIN10/TOCC2/T0/XCK0/SCK"/>
 <wire x1="68.58" y1="2.54" x2="81.28" y2="2.54" width="0.1524" layer="91"/>
 <label x="68.58" y="2.54" size="1.778" layer="95"/>
